File: pcb/Open_TPMX2030.kicad_sch (KiCad schematic)
At the start: 0 parts

Commit message: feat: Adjusting the project for a successful start
Other:
- added sheet keyboard matrix (key_matrix.kicad_sch)
- title: ${PROJECTNAME} -> ${PROJECT_NAME}
Changed lines of the file:
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@@
 	(paper "A4")
 	(title_block
-		(title "${PROJECTNAME}")
+		(title "${PROJECT_NAME}")
 		(date "${CREATION_DATE}")
 		(rev "${REVISION}")
 		(company "${COMPANY}")
-		(comment 1 "${TITLE}")
+		(comment 1 "License: ${LICENSE}")
 		(comment 2 "${USER_EMAIL}")
 		(comment 3 "${USER_NAME}")
 		(comment 4 "Electrical CAD Operator:")
 	)
+	(symbol
+		(lib_id "Artilect-Logo_14x14mm:LOGO")
+		(at 271.78 173.99 0)
+		(unit 1)
+		(body_style 1)
+		(exclude_from_sim no)
+		(in_bom yes)
+		(on_board yes)
+		(in_pos_files yes)
+		(dnp no)
+		(fields_autoplaced yes)
+		(property "Reference" "#G2"
+			(at 271.78 167.6084 0)
+			(hide yes)
+			(show_name no)
+			(do_not_autoplace no)
+			(effects
+				(font
+					(size 1.27 1.27)
+				)
+			)
+		)
+		(property "Value" "LOGO"
+			(at 271.78 180.3716 0)
+			(hide yes)
+			(show_name no)
+			(do_not_autoplace no)
+			(effects
+				(font
+					(size 1.27 1.27)
+				)
+			)
+		)
+		(property "Footprint" ""
+			(at 271.78 173.99 0)
+			(hide yes)
+			(show_name no)
+			(do_not_autoplace no)
+			(effects
+				(font
+					(size 1.27 1.27)
+				)
+			)
+		)
+		(property "Datasheet" ""
+			(at 271.78 173.99 0)
+			(hide yes)
+			(show_name no)
+			(do_not_autoplace no)
+			(effects
+				(font
+					(size 1.27 1.27)
+				)
+			)
+		)
+		(property "Description" ""
+			(at 271.78 173.99 0)
+			(hide yes)
+			(show_name no)
+			(do_not_autoplace no)
+			(effects
+				(font
+					(size 1.27 1.27)
+				)
+			)
+		)
+		(instances
+			(project "Open_TPMX2030"
+				(path "/7eb97883-76c6-4f20-a7ea-f78662082f71"
+					(reference "#G2")
+					(unit 1)
+				)
+			)
+		)
+	)
+	(sheet
+		(at 100.33 68.58)
+		(size 95.25 52.07)
+		(exclude_from_sim no)
+		(in_bom yes)
+		(on_board yes)
+		(dnp no)
+		(fields_autoplaced yes)
+		(stroke
+			(width 0.1524)
+			(type solid)
+		)
+		(fill
+			(color 0 0 0 0)
+		)
+		(property "Sheetname" "keyboard matrix"
+			(at 100.33 67.8684 0)
+			(show_name no)
+			(do_not_autoplace no)
+			(effects
+				(font
+					(size 1.27 1.27)
+				)
+				(justify left bottom)
+			)
+		)
+		(property "Sheetfile" "key_matrix.kicad_sch"
+			(at 100.33 121.2346 0)
+			(show_name no)
+			(do_not_autoplace no)
+			(effects
+				(font
+					(size 1.27 1.27)
+				)
+				(justify left top)
+			)
+		)
+		(instances
+			(project "Open_TPMX2030"
+				(path "/7eb97883-76c6-4f20-a7ea-f78662082f71"
+					(page "2")
+				)
+			)
+		)
+	)
 	(sheet_instances
